Commit message: added nav and moveit launch files

File: moma_description/urdf/ld250_tm12x.urdf (robot description, URDF)
Before this commit: robot ld250_tm12x, 11 links, 10 joints
Links:
- added link laser_frame
Joints:
- added joint base_link_to_laser_frame: type fixed, parent base_link, child laser_frame, origin xyz=0.45 0 0.195

Commit message: updated urdf

File: moma_description/urdf/ld250_tm12x.urdf (robot description, URDF)
Before this commit: robot ld250_tm12x, 12 links, 11 joints
Links:
- removed link main_body
- removed link tm_base
- removed link tm_flange
- removed link tm_link_0
- removed link tm_link_1
- removed link tm_link_2
- removed link tm_link_3
- removed link tm_link_4
- removed link tm_link_5
- removed link tm_link_6
- added link amr_base, mass 4.07; collision mesh filename=package://amr_description/meshes/LD250.obj; visual mesh filename=package://amr_description/meshes/LD250.obj
- added link base
- added link controlbox, mass 4.07; collision mesh filename=package://moma_description/meshes/controlbox/LD250.obj; visual mesh filename=package://moma_description/meshes/controlbox/LD250.obj
- added link flange
- added link link_0, mass 1.0; collision mesh filename=package://tm_description/meshes/tm12/collision/tm12-base_c.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; visual mesh filename=package://tm_description/meshes/tm12/visual/tm12-base.obj
- added link link_1, mass 7.6; collision mesh filename=package://tm_description/meshes/tm12/collision/tmr_750w_01_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; visual mesh filename=package://tm_description/meshes/tm12/visual/tmr_750w_01.obj
- added link link_2, mass 14.0239; collision mesh filename=package://tm_description/meshes/tm12/collision/tm12-arm1_c.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; visual mesh filename=package://tm_description/meshes/tm12/visual/tm12-arm1.obj
- added link link_3, mass 3.3577; collision mesh filename=package://tm_description/meshes/tm12/collision/tm12-arm2_c.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; visual mesh filename=package://tm_description/meshes/tm12/visual/tm12-arm2.obj
- added link link_4, mass 1.576; collision mesh filename=package://tm_description/meshes/tm5-900/collision/tmr_100w_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; visual mesh filename=package://tm_description/meshes/tm5-900/visual/tmr_100w_01.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
- added link link_5, mass 1.576; collision mesh filename=package://tm_description/meshes/tm5-900/collision/tmr_100w_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; visual mesh filename=package://tm_description/meshes/tm5-900/visual/tmr_100w_02.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
- added link link_6, mass 0.31; collision mesh filename=package://tm_description/meshes/tm5-900/collision/tmr_iox_c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; visual mesh filename=package://tm_description/meshes/tm5-900/visual/tmr_iox.obj
Joints:
- removed joint ld250_to_tm12x_mount
- removed joint main_body_to_base
- removed joint tm_base_fixed_joint
- removed joint tm_flange_fixed_joint
- removed joint tm_joint_1
- removed joint tm_joint_2
- removed joint tm_joint_3
- removed joint tm_joint_4
- removed joint tm_joint_5
- removed joint tm_joint_6
- added joint amr_base_to_base_link: type fixed, parent base_link, child amr_base, origin xyz=0 0 0
- added joint base_fixed_joint: type fixed, parent base, child link_0, origin xyz=0.000000 0.000000 0.000000 rpy=0.000000 0.000000 0.000000
- added joint controlbox_to_tm12x_mount: type fixed, parent controlbox, child base, origin xyz=0 0 0.325 rpy=0 0 0
- added joint flange_fixed_joint: type fixed, parent link_6, child flange, origin xyz=0.000000 0.000000 0.000000 rpy=0.000000 0.000000 0.000000
- added joint joint_1: type revolute, parent link_0, child link_1, origin xyz=0.000000 0.000000 0.165200 rpy=0.000000 -0.000000 0.000000, axis 0 0 1, limit lower=-6.283185307179586 upper=6.283185307179586 effort=353 velocity=2.0943951023931953
- added joint joint_2: type revolute, parent link_1, child link_2, origin xyz=0.000000 0.000000 0.000000 rpy=-1.570796 -1.570796 0.000000, axis 0 0 1, limit lower=-6.283185307179586 upper=6.283185307179586 effort=353 velocity=2.0943951023931953
- added joint joint_3: type revolute, parent link_2, child link_3, origin xyz=0.636100 0.000000 0.000000 rpy=0.000000 -0.000000 0.000000, axis 0 0 1, limit lower=-2.897246558310587 upper=2.897246558310587 effort=157 velocity=3.141592653589793
- added joint joint_4: type revolute, parent link_3, child link_4, origin xyz=0.557900 0.000000 -0.156300 rpy=0.000000 -0.000000 1.570796, axis 0 0 1, limit lower=-6.283185307179586 upper=6.283185307179586 effort=54 velocity=3.141592653589793
- added joint joint_5: type revolute, parent link_4, child link_5, origin xyz=0.000000 -0.106000 0.000000 rpy=1.570796 -0.000000 0.000000, axis 0 0 1, limit lower=-6.283185307179586 upper=6.283185307179586 effort=54 velocity=3.141592653589793
- added joint joint_6: type revolute, parent link_5, child link_6, origin xyz=0.000000 -0.113150 0.000000 rpy=1.570796 -0.000000 0.000000, axis 0 0 1, limit lower=-6.283185307179586 upper=6.283185307179586 effort=54 velocity=3.141592653589793
- added joint ld250_to_controlbox: type fixed, parent base_link, child controlbox, origin xyz=0.2 0 0.34 rpy=0 0 0

File: moma_description/xacro/ld250_tm12x.urdf.xacro (robot description, xacro)
@@ -8,4 +8,5 @@
   <xacro:arg name="trans_hw_iface" default="hardware_interface/PositionJointInterface"/>
   <xacro:arg name="arm_base_link" default="base_link"/>
+  <xacro:arg name="controlbox_mesh_pkg" default="moma_description"/>
   <!-- =============================================================== -->
   <!--                   LD250 related configuration                   -->
@@ -44,5 +45,5 @@
       <origin rpy="0 0 3.141582654" xyz="0 0 0"/>
       <geometry>
-        <mesh filename="package://${mesh_pkg}/meshes/controlbox/LD250.obj"/>
+        <mesh filename="package://$(arg controlbox_mesh_pkg)/meshes/controlbox/LD250.obj"/>
       </geometry>
       <material name="white">
@@ -53,5 +54,5 @@
       <origin rpy="0 0 3.141592654" xyz="0 0 0"/>
       <geometry>
-        <mesh filename="package://${mesh_pkg}/meshes/controlbox/LD250.obj"/>
+        <mesh filename="package://$(arg controlbox_mesh_pkg)/meshes/controlbox/LD250.obj"/>
       </geometry>
     </collision>
