Commit message: added new controlbox stl

File: moma_description/xacro/ld250_tm12x.urdf.xacro (robot description, xacro)
@@ -98,5 +98,5 @@
       <origin rpy="0 0 3.141582654" xyz="0 0 0"/>
       <geometry>
-        <mesh filename="package://$(arg controlbox_mesh_pkg)/meshes/controlbox/LD250.obj"/>
+        <mesh filename="package://$(arg controlbox_mesh_pkg)/meshes/controlbox/controlbox.stl"/>
       </geometry>
       <material name="controlbox_white">
@@ -107,5 +107,5 @@
       <origin rpy="0 0 3.141592654" xyz="0 0 0"/>
       <geometry>
-        <mesh filename="package://$(arg controlbox_mesh_pkg)/meshes/controlbox/LD250.obj"/>
+        <mesh filename="package://$(arg controlbox_mesh_pkg)/meshes/controlbox/controlbox.stl"/>
       </geometry>
     </collision>

Commit message: added a proper moveit config for omron_moma and fixed cascading

File: moma_description/xacro/ld250_tm12x.urdf.xacro (robot description, xacro)
@@ -14,4 +14,5 @@
   <!-- Includes -->
   <xacro:include filename="$(find amr_description)/xacro/ld250.urdf.xacro"/>
+  <xacro:include filename="$(find moma_description)/xacro/controlbox_ld250.urdf.xacro"/>
   <!-- LD250 mobile base -->
   <xacro:ld250 prefix="$(arg base_prefix)" mesh_pkg="amr_description"/>
@@ -94,25 +95,5 @@
   <!--             TM12x Control box related configuration             -->
   <!-- =============================================================== -->
-  <link name="controlbox">
-    <visual>
-      <origin rpy="0 0 3.141582654" xyz="0 0 0"/>
-      <geometry>
-        <mesh filename="package://$(arg controlbox_mesh_pkg)/meshes/controlbox/controlbox.stl"/>
-      </geometry>
-      <material name="controlbox_white">
-        <color rgba="1 1 1 1"/>
-      </material>
-    </visual>
-    <collision>
-      <origin rpy="0 0 3.141592654" xyz="0 0 0"/>
-      <geometry>
-        <mesh filename="package://$(arg controlbox_mesh_pkg)/meshes/controlbox/controlbox.stl"/>
-      </geometry>
-    </collision>
-    <inertial>
-      <mass value="4.07"/>
-      <inertia ixx="0.426" ixy="0.0" ixz="0.0" iyy="0.496" iyz="0.0" izz="0.91"/>
-    </inertial>
-  </link>
+  <xacro:controlbox_ld250 mesh_pkg="$(arg controlbox_mesh_pkg)" link_name="controlbox"/>
   <!-- =============================================================== -->
   <!--                Joint Connection configuration                   -->
@@ -122,6 +103,5 @@
     <parent link="$(arg base_prefix)base_link"/>
     <child link="controlbox"/>
-    <!-- <origin xyz="0.2 0 0.34" rpy="0 0 0"/> -->
-    <origin xyz="0 0 0.34" rpy="0 0 0"/>
+    <origin xyz="0 0 0.38" rpy="0 0 0"/>
   </joint>
   <!-- Mount the TM12x base to TM12x control box base -->

Commit message: made the xacro file extendable

File: moma_description/xacro/ld250_tm12x.urdf.xacro (robot description, xacro)
@@ -9,4 +9,5 @@
   <xacro:arg name="arm_base_link" default="base_link"/>
   <xacro:arg name="controlbox_mesh_pkg" default="moma_description"/>
+  <xacro:macro name="ld250_tm12x_robot" params="ns:='' arm_prefix:='' base_prefix:='' arm_color:='none' trans_hw_iface:='hardware_interface/PositionJointInterface' arm_base_link:='base_link' controlbox_mesh_pkg:='moma_description'">
   <!-- =============================================================== -->
   <!--                   LD250 related configuration                   -->
@@ -16,5 +17,5 @@
   <xacro:include filename="$(find moma_description)/xacro/controlbox_ld250.urdf.xacro"/>
   <!-- LD250 mobile base -->
-  <xacro:ld250 prefix="$(arg base_prefix)" mesh_pkg="amr_description"/>
+  <xacro:ld250 prefix="${base_prefix}" mesh_pkg="amr_description"/>
   <!-- =============================================================== -->
   <!--                   TM12x related configuration                   -->
@@ -24,5 +25,5 @@
   <xacro:include filename="$(find tm_description)/xacro/macro.transmission.xacro" />
   <xacro:include filename="$(find tm_description)/xacro/macro.tm12x-nominal.urdf.xacro" />
-  <xacro:property name="arm_color_val" value="$(arg arm_color)"/>
+  <xacro:property name="arm_color_val" value="${arm_color}"/>
   <xacro:property name="tm_effective_arm_color" value="${
     'moma_tm_none' if arm_color_val == 'none' else
@@ -81,19 +82,19 @@
   </material>
   <!-- TM12x arm (gazebo/transmission/material macros) -->
-  <xacro:tmr_gazebo ns="$(arg ns)" prefix="$(arg arm_prefix)" />
-  <xacro:tmr_transmission prefix="$(arg arm_prefix)" hw_iface="$(arg trans_hw_iface)" />
+  <xacro:tmr_gazebo ns="${ns}" prefix="${arm_prefix}" />
+  <xacro:tmr_transmission prefix="${arm_prefix}" hw_iface="${trans_hw_iface}" />
   <!-- TM12x geometry -->
   <!-- If the arm color is 'none' -->
   <xacro:if value="${arm_color_val == 'none'}">
-    <xacro:tm12x ns="$(arg ns)" prefix="$(arg arm_prefix)" color="${tm_effective_arm_color}"/>
+    <xacro:tm12x ns="${ns}" prefix="${arm_prefix}" color="${tm_effective_arm_color}"/>
   </xacro:if>
   <!-- If the arm color is not 'none', include the colored version -->
   <xacro:unless value="${arm_color_val == 'none'}">
-    <xacro:tm12x ns="$(arg ns)" prefix="$(arg arm_prefix)" color="${tm_effective_arm_color}" format="stl"/>
+    <xacro:tm12x ns="${ns}" prefix="${arm_prefix}" color="${tm_effective_arm_color}" format="stl"/>
   </xacro:unless>
   <!-- =============================================================== -->
   <!--             TM12x Control box related configuration             -->
   <!-- =============================================================== -->
-  <xacro:controlbox_ld250 mesh_pkg="$(arg controlbox_mesh_pkg)" link_name="controlbox"/>
+  <xacro:controlbox_ld250 mesh_pkg="${controlbox_mesh_pkg}" link_name="controlbox"/>
   <!-- =============================================================== -->
   <!--                Joint Connection configuration                   -->
@@ -101,5 +102,5 @@
   <!-- Mount the TM12x control box base to the LD250 base_link -->
   <joint name="ld250_to_controlbox" type="fixed">
-    <parent link="$(arg base_prefix)base_link"/>
+    <parent link="${base_prefix}base_link"/>
     <child link="controlbox"/>
     <origin xyz="0 0 0.38" rpy="0 0 0"/>
@@ -108,5 +109,5 @@
   <joint name="controlbox_to_tm12x_mount" type="fixed">
     <parent link="controlbox"/>
-    <child link="$(arg arm_prefix)base"/>
+    <child link="${arm_prefix}base"/>
     <origin xyz="0.2 0 0.325" rpy="0 0 0"/>
   </joint>
@@ -124,3 +125,12 @@
     - control box center to arm base: 198 mm
   -->
+  </xacro:macro>
+  <xacro:ld250_tm12x_robot
+    ns="$(arg ns)"
+    arm_prefix="$(arg arm_prefix)"
+    base_prefix="$(arg base_prefix)"
+    arm_color="$(arg arm_color)"
+    trans_hw_iface="$(arg trans_hw_iface)"
+    arm_base_link="$(arg arm_base_link)"
+    controlbox_mesh_pkg="$(arg controlbox_mesh_pkg)" />
 </robot>

Commit message: turned ld250_tm12x into a macro so that other descriptions can import and extend it

File: moma_description/xacro/ld250_tm12x.urdf.xacro (robot description, xacro)
@@ -9,121 +9,5 @@
   <xacro:arg name="arm_base_link" default="base_link"/>
   <xacro:arg name="controlbox_mesh_pkg" default="moma_description"/>
-  <xacro:macro name="ld250_tm12x_robot" params="ns:='' arm_prefix:='' base_prefix:='' arm_color:='none' trans_hw_iface:='hardware_interface/PositionJointInterface' arm_base_link:='base_link' controlbox_mesh_pkg:='moma_description'">
-  <!-- =============================================================== -->
-  <!--                   LD250 related configuration                   -->
-  <!-- =============================================================== -->
-  <!-- Includes -->
-  <xacro:include filename="$(find amr_description)/xacro/ld250.urdf.xacro"/>
-  <xacro:include filename="$(find moma_description)/xacro/controlbox_ld250.urdf.xacro"/>
-  <!-- LD250 mobile base -->
-  <xacro:ld250 prefix="${base_prefix}" mesh_pkg="amr_description"/>
-  <!-- =============================================================== -->
-  <!--                   TM12x related configuration                   -->
-  <!-- =============================================================== -->
-  <!-- TM12x macro set -->
-  <xacro:include filename="$(find tm_description)/xacro/macro.gazebo.xacro" />
-  <xacro:include filename="$(find tm_description)/xacro/macro.transmission.xacro" />
-  <xacro:include filename="$(find tm_description)/xacro/macro.tm12x-nominal.urdf.xacro" />
-  <xacro:property name="arm_color_val" value="${arm_color}"/>
-  <xacro:property name="tm_effective_arm_color" value="${
-    'moma_tm_none' if arm_color_val == 'none' else
-    'moma_tm_lightgrey' if arm_color_val == 'lightgrey' else
-    'moma_tm_grey' if arm_color_val == 'grey' else
-    'moma_tm_white' if arm_color_val == 'white' else
-    'moma_tm_red' if arm_color_val == 'red' else
-    'moma_tm_orange' if arm_color_val == 'orange' else
-    'moma_tm_yellow' if arm_color_val == 'yellow' else
-    'moma_tm_green' if arm_color_val == 'green' else
-    'moma_tm_blue' if arm_color_val == 'blue' else
-    'moma_tm_indigo' if arm_color_val == 'indigo' else
-    'moma_tm_violet' if arm_color_val == 'violet' else
-    'moma_tm_black' if arm_color_val == 'black' else
-    'moma_tm_darkolive' if arm_color_val == 'darkolive' else
-    arm_color_val
-  }"/>
-  <material name="moma_tm_none">
-    <color rgba="0.0 0.0 0.0 1.0" />
-  </material>
-  <material name="moma_tm_lightgrey">
-    <color rgba="0.5 0.5 0.5 1.0" />
-  </material>
-  <material name="moma_tm_grey">
-    <color rgba="0.75 0.75 0.75 1.0" />
-  </material>
-  <material name="moma_tm_white">
-    <color rgba="0.95 0.95 0.95 1.0" />
-  </material>
-  <material name="moma_tm_red">
-    <color rgba="0.95 0.0 0.0 1.0" />
-  </material>
-  <material name="moma_tm_orange">
-    <color rgba="1.0 0.5 0.0 1.0" />
-  </material>
-  <material name="moma_tm_yellow">
-    <color rgba="1.0 1.0 0.0 1.0" />
-  </material>
-  <material name="moma_tm_green">
-    <color rgba="0.0 1.0 0.0 1.0" />
-  </material>
-  <material name="moma_tm_blue">
-    <color rgba="0.0 0.0 1.0 1.0" />
-  </material>
-  <material name="moma_tm_indigo">
-    <color rgba="0.3 0.3 0.6 1.0" />
-  </material>
-  <material name="moma_tm_violet">
-    <color rgba="0.6 0.0 1.0 1.0" />
-  </material>
-  <material name="moma_tm_black">
-    <color rgba="0.0 0.0 0.0 1.0" />
-  </material>
-  <material name="moma_tm_darkolive">
-    <color rgba="0.3 0.3 0.25 1.0" />
-  </material>
-  <!-- TM12x arm (gazebo/transmission/material macros) -->
-  <xacro:tmr_gazebo ns="${ns}" prefix="${arm_prefix}" />
-  <xacro:tmr_transmission prefix="${arm_prefix}" hw_iface="${trans_hw_iface}" />
-  <!-- TM12x geometry -->
-  <!-- If the arm color is 'none' -->
-  <xacro:if value="${arm_color_val == 'none'}">
-    <xacro:tm12x ns="${ns}" prefix="${arm_prefix}" color="${tm_effective_arm_color}"/>
-  </xacro:if>
-  <!-- If the arm color is not 'none', include the colored version -->
-  <xacro:unless value="${arm_color_val == 'none'}">
-    <xacro:tm12x ns="${ns}" prefix="${arm_prefix}" color="${tm_effective_arm_color}" format="stl"/>
-  </xacro:unless>
-  <!-- =============================================================== -->
-  <!--             TM12x Control box related configuration             -->
-  <!-- =============================================================== -->
-  <xacro:controlbox_ld250 mesh_pkg="${controlbox_mesh_pkg}" link_name="controlbox"/>
-  <!-- =============================================================== -->
-  <!--                Joint Connection configuration                   -->
-  <!-- =============================================================== -->
-  <!-- Mount the TM12x control box base to the LD250 base_link -->
-  <joint name="ld250_to_controlbox" type="fixed">
-    <parent link="${base_prefix}base_link"/>
-    <child link="controlbox"/>
-    <origin xyz="0 0 0.38" rpy="0 0 0"/>
-  </joint>
-  <!-- Mount the TM12x base to TM12x control box base -->
-  <joint name="controlbox_to_tm12x_mount" type="fixed">
-    <parent link="controlbox"/>
-    <child link="${arm_prefix}base"/>
-    <origin xyz="0.2 0 0.325" rpy="0 0 0"/>
-  </joint>
-  <!--
-    Dimensions:
-    - base length: 950 mm
-    - base width: 696 mm
-    - base height: 340 mm
-    - arm base offset front: 175 mm
-    - arm base offset back: 570 mm
-    - arm base offset left: 245 mm
-    - arm base offset right: 250 mm
-    - arm base bottom from ld250 top: 320 mm
-    - control box height: 325 mm
-    - control box center to arm base: 198 mm
-  -->
-  </xacro:macro>
+  <xacro:include filename="$(find moma_description)/xacro/ld250_tm12x_macro.urdf.xacro" />
   <xacro:ld250_tm12x_robot
     ns="$(arg ns)"
